File: tendair.kicad_pcb (KiCad board)
At the start: 2 copper layers, 55 x 26 mm, 18 parts, among them J1 Program, J2 USB_C_Receptacle_PowerOnly_6P, J3 SEN66, Q1 GSBC847BV, U1 ESP32-C3-WROOM-02, U2 AZ1117-3.3

Commit message: stuff
Routing:
- net GND: track 0.00 -> 16.6 mm, vias 0 -> 3
- net /CHIP_PU: track 24.9 -> 31.8 mm, vias 0 -> 2
- added copper zone on B.Cu, net GND
- added copper zone on F.Cu, net GND
Other:
- board text added: "TendAir"
- board text added: "V1"
