File: tendair.kicad_sch (KiCad schematic)
At the start: 16 parts, among them J1 Program, J2 USB_C_Receptacle_PowerOnly_6P, Q1 GSBC847BV, U1 ESP32-C3-WROOM-02, U2 AZ1117-3.3

Commit message: updating the pcb
Parts:
- removed R4: 10k, symbol Device:R_US
- added J3: SEN66, Connector_JST:JST_GH_SM06B-GHS-TB_1x06-1MP_P1.25mm_Horizontal, symbol Connector_Generic:Conn_01x06
- added R7, R8: 10k, Resistor_SMD:R_1206_3216Metric, symbol Device:R_US
- C1, C2, C3, C4, C5: footprint (none) -> Capacitor_SMD:C_1206_3216Metric
- J1: footprint (none) -> Connector_PinHeader_2.54mm:PinHeader_1x06_P2.54mm_Vertical
- Q1: footprint (none) -> Package_TO_SOT_SMD:SOT-563
- R1, R2, R3, R5, R6: footprint (none) -> Resistor_SMD:R_1206_3216Metric
Connections:
- net +3.3V: now also J3.1 (Pin_1), J3.6 (Pin_6), R7.2, R8.2
- net GND: now also J3.2 (Pin_2), J3.5 (Pin_5)
- net GPIO9: now also U1.8 (IO9)
- net SCL: now reaches U1.3 (IO4)
- net SCL: now also J3.4 (Pin_4), R7.1
- net GPIO8 renamed SDA
- net SDA: now also J3.3 (Pin_3), R8.1
- no-connect marks 0 -> 10
Other:
- note added: "IO8 requires a pull-up resistor according to the ESP data sheet. I2C also requires a pullup, so R8 is doing double duty for us."

Commit message: this works well!
Parts:
- J2: URL (none) -> https://www.digikey.com/en/products/detail/amphenol-cs-fci/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
- J3: URL (none) -> https://www.digikey.com/en/products/detail/jst-sales-americ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
- Q1: URL (none) -> https://www.digikey.com/en/products/detail/good-ark-semicon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
- U1: URL (none) -> https://www.digikey.com/en/products/detail/espressif-system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
Changed lines of the file:
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@@
+			)
+		)
+		(property "URL" "https://www.digikey.com/en/products/detail/good-ark-semiconductor/GSBC847BV/24613131"
+			(at 64.77 55.88 0)
+			(effects
+				(font
+					(size 1.27 1.27)
+				)
+				(hide yes)
 			)
 		)
@@
 			)
 		)
+		(property "URL" "https://www.digikey.com/en/products/detail/jst-sales-america-inc/SM06B-GHS-TB/807790"
+			(at 245.11 48.26 0)
+			(effects
+				(font
+					(size 1.27 1.27)
+				)
+				(hide yes)
+			)
+		)
 		(pin "1"
 		)
@@
 		)
 		(property "Description" "USB Power-Only 6P Type-C Receptacle connector"
+			(at 220.98 110.49 0)
+			(effects
+				(font
+					(size 1.27 1.27)
+				)
+				(hide yes)
+			)
+		)
+		(property "URL" "https://www.digikey.com/en/products/detail/amphenol-cs-fci/10164359-00011LF/18443702"
 			(at 220.98 110.49 0)
 			(effects
@@
 			)
 		)
+		(property "URL" "https://www.digikey.com/en/products/detail/good-ark-semiconductor/GSBC847BV/24613131"
+			(at 64.77 76.2 0)
+			(effects
+				(font
+					(size 1.27 1.27)
+				)
+				(hide yes)
+			)
+		)
 		(pin "1"
 		)
@@
 			(effects
 				(font
+					(size 1.27 1.27)
+				)
+				(hide yes)
+			)
+		)
+		(property "URL" "https://www.digikey.com/en/products/detail/espressif-systems/ESP32-C3-WROOM-02-H4/14553033"
+			(at 143.51 132.08 0)
+			(effects
+				(font
